Commit message: added gazebo control

File: description/robot.urdf.xacro (robot description, xacro)
@@ -2,3 +2,4 @@
 <robot xmlns:xacro="http://www.ros.org/wiki/xacro"  name="robot">
 	<xacro:include filename="robot_core_lr.xacro"/>
+	<xacro:include filename="gazebo_control.xacro"/>
 </robot>

File: description/robot_core_lr.xacro (robot description, xacro)
@@ -1,4 +1,5 @@
 <?xml version="1.0"?>
 <robot xmlns:xacro="http://www.ros.org/wiki/xacro">
+	<xacro:include filename="inertial_macros.xacro"/>
 	<material name="white">
 		<color rgba="1 1 1 1"/>
@@ -24,11 +25,25 @@
 			<material name="white"/>
 		</visual>
+		<collision>
+			<origin xyz="0 0 0.1"/>
+			<geometry>
+				<box size="0.8 0.4 0.05"/>
+			</geometry>
+		</collision>
+		<xacro:inertial_box mass="0.5" x="0.8" y="0.4" z="0.05">
+        	<origin xyz="0 0 0.1" rpy="0 0 0"/>
+        </xacro:inertial_box>
 	</link>
+	<gazebo reference="chassis">
+		<material>Gazebo/White</material>
+	</gazebo>
 	<!-- WHEEL1 -->
 	<joint name="wheel1_joint" type="continuous">
 		<parent link="base_link"/>
 		<child link="wheel1_link"/>
-		<origin xyz="0.3 0.25 0" rpy="${-pi/2} 0 0"/>
+		<origin xyz="0.2 0.25 0" rpy="${-pi/2} 0 0"/>
 		<axis xyz="0 0 1"/>
+		<limit effort="10000" velocity="1000" />
+	    <dynamics damping="1.0" friction="1.0" />
 	</joint>
 	<link name="wheel1_link">
@@ -39,11 +54,24 @@
 			<material name="black"/>
 		</visual>
+		<collision>
+			<geometry>
+				<cylinder radius="0.1" length="0.1"/>
+			</geometry>
+		</collision>
+		<xacro:inertial_cylinder mass="0.1" length="0.1" radius="0.1">
+        	<origin xyz="0 0 0" rpy="0 0 0"/>
+        </xacro:inertial_cylinder>
 	</link>
+	<gazebo reference="wheel1_link">
+		<material>Gazebo/Black</material>
+	</gazebo>
 	<!-- WHEEL2 -->
 	<joint name="wheel2_joint" type="continuous">
 		<parent link="base_link"/>
 		<child link="wheel2_link"/>
-		<origin xyz="0.3 -0.25 0" rpy="${pi/2} 0 0"/>
+		<origin xyz="0.2 -0.25 0" rpy="${pi/2} 0 0"/>
 		<axis xyz="0 0 -1"/>
+		<limit effort="10000" velocity="1000" />
+	    <dynamics damping="1.0" friction="1.0" />
 	</joint>
 	<link name="wheel2_link">
@@ -54,11 +82,24 @@
 			<material name="black"/>
 		</visual>
+		<collision>
+			<geometry>
+				<cylinder radius="0.1" length="0.1"/>
+			</geometry>
+		</collision>
+		<xacro:inertial_cylinder mass="0.1" length="0.1" radius="0.1">
+        	<origin xyz="0 0 0" rpy="0 0 0"/>
+        </xacro:inertial_cylinder>
 	</link>
+	<gazebo reference="wheel2_link">
+		<material>Gazebo/Black</material>
+	</gazebo>
 	<!-- WHEEL3 -->
 	<joint name="wheel3_joint" type="continuous">
 		<parent link="base_link"/>
 		<child link="wheel3_link"/>
-		<origin xyz="-0.3 0.25 0" rpy="${-pi/2} 0 0"/>
+		<origin xyz="-0.2 0.25 0" rpy="${-pi/2} 0 0"/>
 		<axis xyz="0 0 1"/>
+		<limit effort="10000" velocity="1000" />
+	    <dynamics damping="1.0" friction="1.0" />
 	</joint>
 	<link name="wheel3_link">
@@ -69,11 +110,24 @@
 			<material name="black"/>
 		</visual>
+		<collision>
+			<geometry>
+				<cylinder radius="0.1" length="0.1"/>
+			</geometry>
+		</collision>
+		<xacro:inertial_cylinder mass="0.1" length="0.1" radius="0.1">
+        	<origin xyz="0 0 0" rpy="0 0 0"/>
+        </xacro:inertial_cylinder>
 	</link>
+	<gazebo reference="wheel3_link">
+		<material>Gazebo/Black</material>
+	</gazebo>
 	<!-- WHEEL4 -->
 	<joint name="wheel4_joint" type="continuous">
 		<parent link="base_link"/>
 		<child link="wheel4_link"/>
-		<origin xyz="-0.3 -0.25 0" rpy="${pi/2} 0 0"/>
+		<origin xyz="-0.2 -0.25 0" rpy="${pi/2} 0 0"/>
 		<axis xyz="0 0 -1"/>
+		<limit effort="10000" velocity="1000" />
+	    <dynamics damping="1.0" friction="1.0" />
 	</joint>
 	<link name="wheel4_link">
@@ -84,4 +138,15 @@
 			<material name="black"/>
 		</visual>
+		<collision>
+			<geometry>
+				<cylinder radius="0.1" length="0.1"/>
+			</geometry>
+		</collision>
+		<xacro:inertial_cylinder mass="0.1" length="0.1" radius="0.1">
+        	<origin xyz="0 0 0" rpy="0 0 0"/>
+        </xacro:inertial_cylinder>
 	</link>
+	<gazebo reference="wheel4_link">
+		<material>Gazebo/Black</material>
+	</gazebo>
 </robot>
